File: wv_esc.sch (KiCad schematic (older format))
At the start: 17 parts, among them J1 Conn_01x02, J3 Conn_01x03, Q7 AS78LXX, U1 ATtiny404-SS

Commit message: use sheet for 5V regulator
Parts:
- removed C7: 0.33μF, 10V, Capacitor_SMD:C_0805_2012Metric, symbol Device:C_Small
- removed C8: 0.1μF, 25V, Capacitor_SMD:C_0805_2012Metric, symbol Device:C_Small
- removed Q7: AS78LXX, Package_TO_SOT_SMD:SOT-89-3, symbol ldos:AS78LXX
- removed U1: ATtiny404-SS, Package_SO:SOIC-14_3.9x8.7mm_P1.27mm, symbol MCU_Microchip_ATtiny:ATtiny404-SS
- added U1: ATtiny204-SS, Package_SO:SOIC-14_3.9x8.7mm_P1.27mm, symbol MCU_Microchip_ATtiny:ATtiny204-SS
- renumbered Comm to Comm1, Debug to Debug1, Sensor to Sensor1
Connections:
- net +5V: now also U1.1 (VCC)
- net GND: now also U1.14 (GND)
- net at Debug1.3 (Pin_3): now also U1.10 (~RESET~/PA0)
- net at R13.2: now also U1.11 (PA1)
- net at R14.2: now also U1.12 (PA2)
- net at R15.2: now also U1.13 (PA3)
- net at Sensor1.3 (Pin_3): now also U1.2 (PA4)
- net at Sensor1.4 (Pin_4): now also U1.3 (PA5)
- net at Sensor1.5 (Pin_5): now also U1.4 (PA6)
- net at R10.2: now also U1.5 (PA7)
- net at Comm1.3 (Pin_3): now also U1.6 (PB3), U1.7 (PB2)
- net at R11.2: now also U1.8 (PB1)
- net at R12.2: now also U1.9 (PB0)
- net +15V renamed 14V
Other:
- moved on the sheet: C5, C6, J1
